Commit message: made rviz visualization for aliengo urdf

File: unitree_gazebo/urdf/aliengo.urdf (robot description, URDF)
Before this commit: robot aliengo, 31 links, 30 joints
Links:
- link FL_calf: geometry collision box size=0.25 0.0208 0.016; visual mesh filename=package://unitree_gazebo/meshes/calf.dae scale=1 1 1
- link FL_hip: geometry collision cylinder length=0.0418 radius=0.046; visual mesh filename=package://unitree_gazebo/meshes/hip.dae scale=1 1 1
- link FL_thigh: geometry collision box size=0.25 0.0374 0.043; visual mesh filename=package://unitree_gazebo/meshes/thigh.dae scale=1 1 1
- link FR_calf: geometry collision box size=0.25 0.0208 0.016; visual mesh filename=package://unitree_gazebo/meshes/calf.dae scale=1 1 1
- link FR_hip: geometry collision cylinder length=0.0418 radius=0.046; visual mesh filename=package://unitree_gazebo/meshes/hip.dae scale=1 1 1
- link FR_thigh: geometry collision box size=0.25 0.0374 0.043; visual mesh filename=package://unitree_gazebo/meshes/thigh_mirror.dae scale=1 1 1
- link RL_calf: geometry collision box size=0.25 0.0208 0.016; visual mesh filename=package://unitree_gazebo/meshes/calf.dae scale=1 1 1
- link RL_hip: geometry collision cylinder length=0.0418 radius=0.046; visual mesh filename=package://unitree_gazebo/meshes/hip.dae scale=1 1 1
- link RL_thigh: geometry collision box size=0.25 0.0374 0.043; visual mesh filename=package://unitree_gazebo/meshes/thigh.dae scale=1 1 1
- link RR_calf: geometry collision box size=0.25 0.0208 0.016; visual mesh filename=package://unitree_gazebo/meshes/calf.dae scale=1 1 1
- link RR_hip: geometry collision cylinder length=0.0418 radius=0.046; visual mesh filename=package://unitree_gazebo/meshes/hip.dae scale=1 1 1
- link RR_thigh: geometry collision box size=0.25 0.0374 0.043; visual mesh filename=package://unitree_gazebo/meshes/thigh_mirror.dae scale=1 1 1
- link trunk: geometry collision box size=0.647 0.15 0.112; visual mesh filename=package://unitree_gazebo/meshes/trunk.dae scale=1 1 1
